File: RSC_Lite_Upgrade_Mod.kicad_pcb (KiCad board)
At the start: 2 copper layers, 36.8 x 48 mm, 30 parts, among them J1 USB_B_Micro, J2 Boot Mode, J3 SWD, J4 JTAG, SW1 RESET, U1 STM32F103C8Tx, Y1 8Mhz

Commit message: Update pcb
Routing:
- net GND: track 262.1 -> 270.4 mm, vias 7 -> 10
- added copper zone on B.Cu, net GND
- added copper zone on F.Cu, net GND
Changed lines of the file:
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@@
 		(tags "Through hole angled pin header THT 1x06 2.54mm single row")
 		(property "Reference" "J4"
-			(at 4.385 -2.27 360)
+			(at 2.794 -2.54 180)
 			(layer "F.SilkS")
 			(effects
@@
 	)
 	(segment
-		(start 185.5055 49.53)
-		(end 185.5055 45.6345)
-		(width 0.4)
-		(layer "F.Cu")
-		(net 2)
-	)
-	(segment
 		(start 196.952646 66.098736)
 		(end 196.38591 65.532)
@@
 	)
 	(segment
+		(start 185.5055 42.5035)
+		(end 184.404 41.402)
+		(width 0.4)
+		(layer "F.Cu")
+		(net 2)
+	)
+	(segment
 		(start 206.756 43.688)
 		(end 206.756 44.196)
@@
 	)
 	(segment
+		(start 185.5055 49.53)
+		(end 185.5055 46.482)
+		(width 0.4)
+		(layer "F.Cu")
+		(net 2)
+	)
+	(segment
 		(start 199.952646 77.524646)
 		(end 199.952646 75.193646)
@@
 	)
 	(segment
+		(start 185.5055 46.482)
+		(end 185.5055 42.5035)
+		(width 0.4)
+		(layer "F.Cu")
+		(net 2)
+	)
+	(segment
 		(start 193.548 74.003382)
 		(end 193.548 74.168)
@@
 	)
 	(segment
+		(start 185.5055 46.482)
+		(end 185.5055 45.6345)
+		(width 0.4)
+		(layer "F.Cu")
+		(net 2)
+	)
+	(segment
 		(start 204.901708 68.326)
 		(end 206.590854 66.636854)
@@
 	)
 	(via
+		(at 184.404 41.402)
+		(size 0.6)
+		(drill 0.3)
+		(layers "F.Cu" "B.Cu")
+		(free yes)
+		(net 2)
+	)
+	(via
 		(at 199.9365 60.198)
 		(size 0.6)
@@
 		(net 2)
 	)
+	(via
+		(at 184.404 85.852)
+		(size 0.6)
+		(drill 0.3)
+		(layers "F.Cu" "B.Cu")
+		(free yes)
+		(net 2)
+	)
+	(via
+		(at 217.678 85.852)
+		(size 0.6)
+		(drill 0.3)
+		(layers "F.Cu" "B.Cu")
+		(free yes)
+		(net 2)
+	)
 	(segment
 		(start 199.39 61.722)
@@
 	)
 	(segment
+		(start 217.805 85.217)
+		(end 217.805 85.725)
+		(width 0.4)
+		(layer "B.Cu")
+		(net 2)
+	)
+	(segment
 		(start 211.608 52.971)
 		(end 211.215 52.578)
@@
 	)
 	(segment
+		(start 185.968 85.852)
+		(end 186.202 85.618)
+		(width 0.4)
+		(layer "B.Cu")
+		(net 2)
+	)
+	(segment
 		(start 201.676 86.36)
 		(end 209.042 86.36)
@@
 	)
 	(segment
+		(start 217.805 85.725)
+		(end 217.678 85.852)
+		(width 0.4)
+		(layer "B.Cu")
+		(net 2)
+	)
+	(segment
+		(start 184.404 85.852)
+		(end 185.968 85.852)
+		(width 0.4)
+		(layer "B.Cu")
+		(net 2)
+	)
+	(segment
 		(start 186.944 86.36)
 		(end 201.676 86.36)
@@
 	(segment
 		(start 217.932 85.09)
+		(end 217.805 85.217)
+		(width 0.4)
+		(layer "B.Cu")
+		(net 2)
+	)
+	(segment
+		(start 217.932 85.09)
 		(end 217.932 74.168)
 		(width 0.4)
@@
 		(net 51)
 	)
+	(zone
+		(net 2)
+		(net_name "GND")
+		(layers "F&B.Cu")
+		(hatch edge 0.5)
+		(connect_pads
+			(clearance 0.5)
+		)
+		(min_thickness 0.25)
+		(filled_areas_thickness no)
+		(fill yes
+			(thermal_gap 0.5)
+			(thermal_bridge_width 0.5)
+		)
+		(polygon
+			(pts
+				(xy 180.34 38.1) (xy 220.98 38.1) (xy 220.98 88.9) (xy 180.34 88.9)
+			)
+		)
+	)
 )

Commit message: Update the PCB
Routing:
- net GND: track 270.4 -> 326.5 mm, vias 10 -> 20
Other:
- outline, holes or cut-outs redrawn
- board text added: "BOOT0"
- board text added: "BOOT1"
- board text added: "GND"
- board text added: "RSC Lite FW Upgrader"
- board text added: "Rev.0"
- board text added: "SWCLK"
- board text added: "SWDIO"
- board text added: "TCK"
- board text added: "TDI"
- board text added: "TDO"
- board text added: "TMS"
- board text added: "VCC"

Commit message: add another gnd via
Routing:
- net GND: track 326.5 -> 331.1 mm, vias 20 -> 21
Changed lines of the file:
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@@
+	)
+	(via
+		(at 194.056 59.944)
+		(size 0.6)
+		(drill 0.3)
+		(layers "F.Cu" "B.Cu")
+		(free yes)
+		(net 2)
 	)
 	(via
@@
 	)
 	(segment
+		(start 194.056 59.944)
+		(end 194.398854 60.286854)
+		(width 0.4)
+		(layer "B.Cu")
+		(net 2)
+	)
+	(segment
 		(start 197.104 62.738)
 		(end 197.612 62.738)
@@
 		(width 0.4)
 		(layer "B.Cu")
+		(net 2)
+	)
+	(segment
+		(start 194.398854 60.286854)
+		(end 194.398854 64.427146)
+		(width 0.4)
+		(layer "B.Cu")
