File: RSC_Lite_Upgrade_Mod.kicad_pcb (KiCad board)
At the start: 2 copper layers, 36.8 x 48 mm, 30 parts, among them J1 USB_B_Micro, J2 Boot Mode, J3 SWD, J4 JTAG, SW1 RESET, U1 STM32F103C8Tx, Y1 8Mhz

Commit message: Update PCB layout
Routing:
- net GND: track 331.1 -> 324.0 mm, vias 21 -> 22
- net VCC: track 155.5 -> 152.1 mm, vias 10 -> 8
Other:
- outline, holes or cut-outs redrawn
Changed lines of the file:
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@@
 		(tags "resistor array")
 		(property "Reference" "RN2"
-			(at 0 -2.8 0)
+			(at 0.1035 -2.806 0)
 			(layer "F.SilkS")
 			(effects
@@
 		)
 		(property "Value" "10K"
-			(at 0 2.8 0)
+			(at 0.1035 2.794 0)
 			(layer "F.SilkS")
 			(effects
@@
 		(layer "B.SilkS")
 	)
+	(gr_line
+		(start 183.388 69.6595)
+		(end 183.388 85.4075)
+		(stroke
+			(width 0.05)
+			(type default)
+		)
+		(layer "Edge.Cuts")
+	)
 	(gr_arc
 		(start 219.456 85.884)
@@
 	)
 	(gr_line
+		(start 182.626 69.2785)
+		(end 183.388 69.6595)
+		(stroke
+			(width 0.05)
+			(type default)
+		)
+		(layer "Edge.Cuts")
+	)
+	(gr_line
 		(start 217.456 87.884)
 		(end 184.626 87.884)
@@
 	)
 	(gr_line
+		(start 182.626 85.7885)
+		(end 182.626 85.884)
+		(stroke
+			(width 0.05)
+			(type default)
+		)
+		(layer "Edge.Cuts")
+	)
+	(gr_line
+		(start 183.388 85.4075)
+		(end 182.626 85.7885)
+		(stroke
+			(width 0.05)
+			(type default)
+		)
+		(layer "Edge.Cuts")
+	)
+	(gr_line
 		(start 188.595 40.894)
 		(end 188.595 40.132)
@@
 	)
 	(gr_line
-		(start 182.626 85.884)
+		(start 182.626 69.2785)
 		(end 182.626 41.878)
 		(stroke
@@
 		(layer "Edge.Cuts")
 	)
+	(gr_text "Rev.0"
+		(at 185.801 41.529 0)
+		(layer "F.Cu")
+		(effects
+			(font
+				(size 1 1)
+				(thickness 0.1)
+			)
+		)
+	)
+	(gr_text "RSC Lite FW Upgrader"
+		(at 183.769 48.641 90)
+		(layer "F.Cu")
+		(effects
+			(font
+				(size 0.7 0.7)
+				(thickness 0.14)
+				(bold yes)
+			)
+		)
+	)
 	(gr_text "GND"
 		(at 185.928 65.532 0)
@@
 		)
 	)
-	(gr_text "Rev.0"
-		(at 185.801 41.529 0)
-		(layer "F.SilkS")
+	(gr_text "RSC Lite FW Upgrader"
+		(at 183.769 48.641 90)
+		(layer "F.Mask")
 		(effects
 			(font
-				(size 1 1)
-				(thickness 0.1)
+				(size 0.7 0.7)
+				(thickness 0.14)
+				(bold yes)
 			)
 		)
 	)
-	(gr_text "RSC Lite FW Upgrader"
-		(at 184.023 48.641 90)
-		(layer "F.SilkS")
+	(gr_text "Rev.0"
+		(at 185.801 41.529 0)
+		(layer "F.Mask")
 		(effects
 			(font
-				(size 0.7 0.7)
-				(thickness 0.14)
-				(bold yes)
+				(size 1 1)
+				(thickness 0.1)
 			)
 		)
@@
 	)
 	(segment
+		(start 186.374 44.131)
+		(end 186.436 44.069)
+		(width 0.4)
+		(layer "F.Cu")
+		(net 2)
+	)
+	(segment
 		(start 210.065 42.0049)
 		(end 208.4391 42.0049)
@@
 	)
 	(segment
+		(start 200.914 42.418)
+		(end 193.04 42.418)
+		(width 0.4)
+		(layer "F.Cu")
+		(net 2)
+	)
+	(segment
 		(start 209.804 79.502)
 		(end 205.816292 79.502)
@@
 	)
 	(segment
+		(start 188.976 42.418)
+		(end 193.04 42.418)
+		(width 0.4)
+		(layer "F.Cu")
+		(net 2)
+	)
+	(segment
 		(start 188.8495 45.316)
 		(end 199.39 45.316)
@@
 	)
 	(segment
-		(start 185.5055 42.5035)
-		(end 184.404 41.402)
+		(start 206.756 43.688)
+		(end 206.756 44.196)
 		(width 0.4)
 		(layer "F.Cu")
@@
 	)
 	(segment
-		(start 206.756 43.688)
-		(end 206.756 44.196)
+		(start 186.374 44.766)
+		(end 188.2995 44.766)
 		(width 0.4)
 		(layer "F.Cu")
@@
 	)
 	(segment
-		(start 186.374 44.766)
-		(end 188.2995 44.766)
+		(start 188.2995 43.0945)
+		(end 188.976 42.418)
 		(width 0.4)
 		(layer "F.Cu")
@@
 	)
 	(segment
-		(start 206.7175 44.2345)
-		(end 206.7175 46.228)
+		(start 186.374 44.766)
+		(end 186.374 44.131)
 		(width 0.4)
 		(layer "F.Cu")
@@
 	)
 	(segment
-		(start 185.5055 46.482)
-		(end 185.5055 42.5035)
+		(start 206.7175 44.2345)
+		(end 206.7175 46.228)
 		(width 0.4)
 		(layer "F.Cu")
@@
 	)
 	(segment
+		(start 188.2995 44.766)
+		(end 188.341 44.8075)
+		(width 0.4)
+		(layer "F.Cu")
+		(net 2)
+	)
+	(segment
 		(start 217.215 44.405)
 		(end 216.8651 44.7549)
@@
 	)
 	(segment
+		(start 188.2995 44.766)
+		(end 188.2995 43.0945)
+		(width 0.4)
+		(layer "F.Cu")
+		(net 2)
+	)
+	(segment
 		(start 209.042 82.296)
 		(end 209.042 86.36)
@@
 	)
 	(via
+		(at 188.2995 44.766)
+		(size 0.6)
+		(drill 0.3)
+		(layers "F.Cu" "B.Cu")
+		(net 2)
+	)
+	(via
 		(at 197.104 62.738)
 		(size 0.6)
@@
 	)
 	(via
-		(at 184.404 41.402)
+		(at 186.436 44.069)
 		(size 0.6)
 		(drill 0.3)
 		(layers "F.Cu" "B.Cu")
-		(free yes)
 		(net 2)
 	)
@@
 	)
 	(segment
-		(start 200.914 42.418)
-		(end 185.42 42.418)
-		(width 0.4)
-		(layer "B.Cu")
-		(net 2)
-	)
-	(segment
 		(start 211.608 52.971)
 		(end 211.215 52.578)
@@
 	)
 	(segment
-		(start 185.42 42.418)
-		(end 184.404 41.402)
-		(width 0.4)
-		(layer "B.Cu")
-		(net 2)
-	)
-	(segment
 		(start 192.189146 71.565196)
 		(end 192.189146 75.857146)
@@
 	)
 	(segment
-		(start 184.658 83.82)
-		(end 187.452 83.82)
-		(width 0.4)
-		(layer "F.Cu")
-		(net 5)
-	)
-	(segment
 		(start 203.454 66.294)
 		(end 203.454 66.802)
@@
 	)
 	(segment
-		(start 183.426 82.57)
-		(end 183.426 82.588)
-		(width 0.4)
-		(layer "F.Cu")
-		(net 5)
-	)
-	(segment
 		(start 203.454 66.802)
 		(end 203.365146 66.890854)
@@
 	)
 	(segment
+		(start 187.452 83.82)
+		(end 184.658 81.026)
+		(width 0.4)
+		(layer "F.Cu")
+		(net 5)
+	)
+	(segment
+		(start 183.408 66.675)
+		(end 183.408 59.172)
+		(width 0.4)
+		(layer "F.Cu")
+		(net 5)
+	)
+	(segment
+		(start 183.408 59.172)
+		(end 184.658 57.922)
+		(width 0.4)
+		(layer "F.Cu")
+		(net 5)
+	)
+	(segment
 		(start 192.189146 66.636854)
 		(end 192.189146 63.665146)
@@
 	)
 	(segment
-		(start 183.426 82.588)
-		(end 184.658 83.82)
+		(start 184.658 81.026)
+		(end 184.658 67.925)
 		(width 0.4)
 		(layer "F.Cu")
@@
 	)
 	(segment
+		(start 184.658 67.925)
+		(end 183.408 66.675)
+		(width 0.4)
+		(layer "F.Cu")
+		(net 5)
+	)
+	(segment
 		(start 200.914 77.216)
 		(end 200.452646 76.754646)
@@
 	)
 	(via
-		(at 184.658 83.82)
-		(size 0.6)
-		(drill 0.3)
-		(layers "F.Cu" "B.Cu")
-		(net 5)
-	)
-	(via
 		(at 192.189146 66.636854)
 		(size 0.6)
@@
 		(net 5)
 	)
-	(via
-		(at 183.426 82.57)
-		(size 0.6)
-		(drill 0.3)
-		(layers "F.Cu" "B.Cu")
-		(net 5)
-	)
 	(segment
 		(start 209.804 69.342)
@@
 	)
 	(segment
-		(start 184.658 57.922)
-		(end 183.408 59.172)
-		(width 0.4)
-		(layer "B.Cu")
-		(net 5)
-	)
-	(segment
 		(start 204.800292 64.008)
 		(end 204.381146 64.427146)
@@
 	)
 	(segment
-		(start 183.408 82.57)
-		(end 183.426 82.57)
-		(width 0.4)
-		(layer "B.Cu")
-		(net 5)
-	)
-	(segment
 		(start 212.09 69.342)
 		(end 209.804 69.342)
@@
 	)
 	(segment
-		(start 183.408 59.172)
-		(end 183.408 82.57)
-		(width 0.4)
-		(layer "B.Cu")
-		(net 5)
-	)
-	(segment
 		(start 191.77 63.246)
 		(end 191.77 58.14)
@@
 	)
 	(segment
-		(start 183.408 82.57)
-		(end 184.658 83.82)
-		(width 0.4)
-		(layer "B.Cu")
-		(net 5)
-	)
-	(segment
 		(start 210.99 84.712)
 		(end 210.82 84.882)
@@
 			)
 		)
+	)
+	(zone
+		(net 0)
+		(net_name "")
+		(layers "F.Cu" "Edge.Cuts")
+		(hatch edge 0.5)
+		(connect_pads
+			(clearance 0)
+		)
+		(min_thickness 0.25)
+		(filled_areas_thickness no)
+		(keepout
+			(tracks allowed)
+			(vias allowed)
+			(pads allowed)
+			(copperpour not_allowed)
+			(footprints allowed)
+		)
+		(fill
+			(thermal_gap 0.5)
+			(thermal_bridge_width 0.5)
+		)
+		(polygon
+			(pts
+				(xy 181.102 39.116) (xy 188.341 39.116) (xy 188.341 42.545) (xy 181.102 42.545)
+			)
+		)

Commit message: Move some traces around
Routing:
- net GND: track 324.0 -> 348.9 mm, vias 22 -> 26
- net /SWDIO: track 18.7 -> 18.0 mm
Changed lines of the file:
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@@
-	)
-	(segment
-		(start 199.99 73.411471)
-		(end 199.99 75.156292)
-		(width 0.2)
-		(layer "F.Cu")
-		(net 2)
 	)
 	(segment
@@
 	)
 	(segment
+		(start 199.99 73.411471)
+		(end 199.638529 73.06)
+		(width 0.2)
+		(layer "F.Cu")
+		(net 2)
+	)
+	(segment
 		(start 210.82 81.782)
 		(end 209.556 81.782)
@@
 	)
 	(segment
+		(start 195.961 73.281146)
+		(end 195.040146 73.281146)
+		(width 0.2)
+		(layer "F.Cu")
+		(net 2)
+	)
+	(segment
 		(start 211.8686 45.4085)
 		(end 211.215 44.7549)
@@
 	)
 	(segment
-		(start 198.920325 73.281146)
-		(end 199.141471 73.06)
-		(width 0.2)
-		(layer "F.Cu")
-		(net 2)
-	)
-	(segment
 		(start 211.239146 66.636854)
 		(end 206.590854 66.636854)
@@
 	)
 	(segment
+		(start 196.182146 73.06)
+		(end 195.961 73.281146)
+		(width 0.2)
+		(layer "F.Cu")
+		(net 2)
+	)
+	(segment
 		(start 199.9365 56.9345)
 		(end 199.3495 56.3475)
@@
 	)
 	(segment
-		(start 199.141471 73.06)
-		(end 199.638529 73.06)
-		(width 0.2)
-		(layer "F.Cu")
-		(net 2)
-	)
-	(segment
 		(start 206.7175 49.53)
 		(end 206.7175 52.07)
@@
 	)
 	(segment
-		(start 199.99 75.156292)
-		(end 199.952646 75.193646)
+		(start 199.638529 73.06)
+		(end 196.182146 73.06)
 		(width 0.2)
 		(layer "F.Cu")
@@
 	)
 	(segment
-		(start 199.638529 73.06)
-		(end 199.99 73.411471)
-		(width 0.2)
-		(layer "F.Cu")
-		(net 2)
-	)
-	(segment
 		(start 208.4391 42.0049)
 		(end 206.756 43.688)
@@
 	)
 	(segment
+		(start 201.549 73.533)
+		(end 201.549 68.58)
+		(width 0.4)
+		(layer "F.Cu")
+		(net 2)
+	)
+	(segment
 		(start 211.215 44.7549)
 		(end 210.6169 44.7549)
@@
 	)
 	(segment
+		(start 199.99 75.156292)
+		(end 199.99 73.411471)
+		(width 0.2)
+		(layer "F.Cu")
+		(net 2)
+	)
+	(segment
 		(start 194.270236 73.281146)
 		(end 193.548 74.003382)
@@
 	)
 	(segment
-		(start 195.040146 73.281146)
-		(end 198.920325 73.281146)
-		(width 0.2)
-		(layer "F.Cu")
-		(net 2)
-	)
-	(segment
 		(start 185.5055 49.53)
 		(end 185.5055 52.07)
@@
 	)
 	(segment
+		(start 199.952646 75.193646)
+		(end 199.99 75.156292)
+		(width 0.2)
+		(layer "F.Cu")
+		(net 2)
+	)
+	(segment
 		(start 204.901708 68.326)
 		(end 206.590854 66.636854)
@@
 	)
 	(via
+		(at 201.549 68.58)
+		(size 0.6)
+		(drill 0.3)
+		(layers "F.Cu" "B.Cu")
+		(free yes)
+		(net 2)
+	)
+	(via
 		(at 193.04 42.418)
 		(size 0.6)
@@
 	)
 	(via
+		(at 201.549 73.533)
+		(size 0.6)
+		(drill 0.3)
+		(layers "F.Cu" "B.Cu")
+		(free yes)
+		(net 2)
+	)
+	(via
 		(at 199.9365 57.912)
 		(size 0.6)
@@
 	)
 	(via
+		(at 196.85 73.533)
+		(size 0.6)
+		(drill 0.3)
+		(layers "F.Cu" "B.Cu")
+		(free yes)
+		(net 2)
+	)
+	(via
 		(at 199.9365 60.198)
 		(size 0.6)
@@
 	(via
 		(at 217.678 85.852)
+		(size 0.6)
+		(drill 0.3)
+		(layers "F.Cu" "B.Cu")
+		(free yes)
+		(net 2)
+	)
+	(via
+		(at 196.85 68.58)
 		(size 0.6)
 		(drill 0.3)
@@
 	)
 	(segment
+		(start 196.85 68.58)
+		(end 191.389 68.58)
+		(width 0.4)
+		(layer "B.Cu")
+		(net 2)
+	)
+	(segment
 		(start 197.104 77.724)
 		(end 196.85 77.47)
@@
 	)
 	(segment
+		(start 191.262 68.453)
+		(end 191.262 70.63805)
+		(width 0.4)
+		(layer "B.Cu")
+		(net 2)
+	)
+	(segment
 		(start 211.215 52.578)
 		(end 211.215 44.7549)
@@
 	)
 	(segment
+		(start 200.722 74.36)
+		(end 197.677 74.36)
+		(width 0.4)
+		(layer "B.Cu")
+		(net 2)
+	)
+	(segment
 		(start 192.189146 71.565196)
 		(end 192.189146 75.857146)
@@
 	)
 	(segment
+		(start 201.549 73.533)
+		(end 200.722 74.36)
+		(width 0.4)
+		(layer "B.Cu")
+		(net 2)
+	)
+	(segment
+		(start 197.677 74.36)
+		(end 196.85 73.533)
+		(width 0.4)
+		(layer "B.Cu")
+		(net 2)
+	)
+	(segment
+		(start 191.389 68.58)
+		(end 191.262 68.453)
+		(width 0.4)
+		(layer "B.Cu")
+		(net 2)
+	)
+	(segment
 		(start 196.938854 64.427146)
 		(end 194.398854 64.427146)
@@
 	)
 	(segment
+		(start 201.549 73.533)
+		(end 201.549 77.597)
+		(width 0.4)
+		(layer "B.Cu")
+		(net 2)
+	)
+	(segment
 		(start 185.968 85.852)
 		(end 186.202 85.618)
@@
 	)
 	(segment
+		(start 201.549 68.58)
+		(end 196.85 68.58)
+		(width 0.4)
+		(layer "B.Cu")
+		(net 2)
+	)
+	(segment
 		(start 187.794854 64.427146)
 		(end 188.595 64.427146)
@@
 	)
 	(segment
-		(start 191.262 64.427146)
-		(end 191.262 70.63805)
-		(width 0.4)
-		(layer "B.Cu")
-		(net 2)
-	)
-	(segment
 		(start 217.118 73.354)
 		(end 214.884 73.354)
@@
 	)
 	(segment
+		(start 191.262 64.427146)
+		(end 191.262 68.453)
+		(width 0.4)
+		(layer "B.Cu")
+		(net 2)
+	)
+	(segment
 		(start 186.68 65.542)
 		(end 187.794854 64.427146)
@@
 	)
 	(segment
+		(start 201.549 77.597)
+		(end 201.422 77.724)
+		(width 0.4)
+		(layer "B.Cu")
+		(net 2)
+	)
+	(segment
 		(start 211.608 59.944)
 		(end 211.608 52.971)
@@
 	)
 	(segment
-		(start 191.516 59.528)
-		(end 192.278 60.29)
-		(width 0.2)
-		(layer "F.Cu")
-		(net 13)
-	)
-	(segment
-		(start 188.91 59.528)
-		(end 191.516 59.528)
-		(width 0.2)
-		(layer "F.Cu")
-		(net 13)
-	)
-	(segment
 		(start 184.674 60.478)
 		(end 184.658 60.462)
@@
 	)
 	(segment
-		(start 195.58 62.738)
-		(end 195.961 63.119)
+		(start 197.452646 65.753646)
+		(end 194.437 62.738)
 		(width 0.2)
 		(layer "F.Cu")
@@
 	)
 	(segment
+		(start 188.91 59.528)
+		(end 187.96 60.478)
+		(width 0.2)
+		(layer "F.Cu")
+		(net 13)
+	)
+	(segment
+		(start 192.278 60.29)
+		(end 191.516 59.528)
+		(width 0.2)
+		(layer "F.Cu")
+		(net 13)
+	)
+	(segment
+		(start 194.437 62.738)
+		(end 192.786 62.738)
+		(width 0.2)
+		(layer "F.Cu")
+		(net 13)
+	)
+	(segment
+		(start 191.516 59.528)
+		(end 188.91 59.528)
+		(width 0.2)
+		(layer "F.Cu")
+		(net 13)
+	)
+	(segment
 		(start 192.786 62.738)
-		(end 195.58 62.738)
+		(end 192.278 62.23)
 		(width 0.2)
 		(layer "F.Cu")
@@
 	)
 	(segment
-		(start 192.278 60.29)
-		(end 192.278 62.23)
+		(start 192.278 62.23)
+		(end 192.278 60.29)
 		(width 0.2)
 		(layer "F.Cu")
@@
 	)
 	(segment
-		(start 197.452646 64.610646)
-		(end 195.961 63.119)
-		(width 0.2)
-		(layer "F.Cu")
-		(net 13)
-	)
-	(segment
-		(start 192.278 62.23)
-		(end 192.786 62.738)
-		(width 0.2)
-		(layer "F.Cu")
-		(net 13)
-	)
-	(segment
-		(start 187.96 60.478)
-		(end 188.91 59.528)
-		(width 0.2)
-		(layer "F.Cu")
-		(net 13)
-	)
-	(segment
 		(start 197.452646 66.868646)
-		(end 197.452646 64.610646)
-		(width 0.2)
-		(layer "F.Cu")
+		(end 197.452646 65.753646)
+		(width 0.2)
+		(layer "F.Cu")
