File: RSC_Lite_Upgrade_Mod.kicad_sch (KiCad schematic)
At the start: 22 parts, among them J3 SWD, J4 JTAG, U1 STM32F103C8Tx, Y1 8Mhz

Commit message: Some more rerouting
Parts:
- U1: value STM32F103C8Tx -> 32F103C8T6
Changed lines of the file:
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@@
 			)
 		)
-		(property "Value" "STM32F103C8Tx"
+		(property "Value" "32F103C8T6"
 			(at 131.7341 125.73 0)
 			(effects

Commit message: Reorganize REV.2 board
Connections:
- net GND: now also J4.5 (Pin_5); no longer J4.2 (Pin_2)
- net JTAG_TCK: now also J4.3 (Pin_3); no longer J4.4 (Pin_4)
- net JTAG_TDI: now also J4.2 (Pin_2); no longer J4.5 (Pin_5)
- net JTAG_TDO: now also J4.4 (Pin_4); no longer J4.3 (Pin_3)
- net JTAG_TMS: now also J4.1 (Pin_1); no longer J4.6 (Pin_6)
- net VCC: now also J4.6 (Pin_6); no longer J4.1 (Pin_1)
Changed lines of the file:
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@@
 	(symbol
 		(lib_id "Connector:Conn_01x06_Pin")
-		(at 233.68 147.32 0)
+		(at 233.68 149.86 0)
+		(mirror x)
 		(unit 1)
 		(exclude_from_sim no)
@@
 		(on_board yes)
 		(dnp no)
-		(fields_autoplaced yes)
 		(property "Reference" "J4"
-			(at 234.315 137.16 0)
+			(at 234.315 160.02 0)
 			(effects
 				(font
@@
 		)
 		(property "Value" "JTAG"
-			(at 234.315 139.7 0)
+			(at 234.315 157.48 0)
 			(effects
 				(font
@@
 		)
 		(property "Footprint" "Connector_PinHeader_2.54mm:PinHeader_1x06_P2.54mm_Horizontal"
-			(at 233.68 147.32 0)
+			(at 233.68 149.86 0)
 			(effects
 				(font
@@
 		)
 		(property "Datasheet" "~"
-			(at 233.68 147.32 0)
+			(at 233.68 149.86 0)
 			(effects
 				(font
@@
 		)
 		(property "Description" "Generic connector, single row, 01x06, script generated"
-			(at 233.68 147.32 0)
+			(at 233.68 149.86 0)
 			(effects
 				(font
